File: output/pcbs/board.kicad_pcb (KiCad board)
At the start: 2 copper layers, 139.1 x 103.9 mm, 46 parts, among them J1 Jumper, J2 Jumper

Commit message: completed routing
Routing:
- net col_pinky: track 0.00 -> 180.8 mm, vias 0 -> 5
- net col_middle: track 0.00 -> 178.2 mm, vias 0 -> 7
- net col_index: track 0.00 -> 171.6 mm, vias 0 -> 6
- net row_top: track 0.00 -> 168.1 mm, vias 0 -> 2
- net row_bottom: track 0.00 -> 163.0 mm, vias 0 -> 1
- net row_home: track 0.00 -> 162.3 mm, vias 0 -> 2
- net col_ring: track 0.00 -> 156.2 mm, vias 0 -> 5
- net col_inner: track 0.00 -> 153.1 mm, vias 0 -> 4
- net row_thumb: track 0.00 -> 114.4 mm, vias 0 -> 4
- net GND: track 0.00 -> 101.3 mm, vias 0 -> 1
- net RAW: track 0.00 -> 93.6 mm, vias 0 -> 2
- net P0: track 0.00 -> 84.8 mm, vias 0 -> 1
- net RST: track 0.00 -> 77.5 mm
- net VCC: track 0.00 -> 76.0 mm, vias 0 -> 1
- net Bplus: track 0.00 -> 62.5 mm, vias 0 -> 3
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Other:
- outline, holes or cut-outs redrawn
